File: troll_cup/PCB/PCB.kicad_sch (KiCad schematic)
At the start: 9 parts, among them SW1 SW_Push, SW2 SW_Push, U1 ATtiny85-20P, U2 DFPLAYER MINI

Commit message: Organize schematic
Parts:
- removed BT1: Battery_Cell, symbol Device:Battery_Cell
- removed LS1: Speaker, symbol Device:Speaker
- added BAT1: TO_BATTERY, Connector_JST:JST_PH_S2B-PH-K_1x02_P2.00mm_Horizontal, symbol Connector_Generic:Conn_01x02
- added SPK1: ~, Connector_JST:JST_PH_S2B-PH-K_1x02_P2.00mm_Horizontal, symbol Connector_Generic:Conn_01x02
- C1: footprint (none) -> Capacitor_SMD:C_0603_1608Metric_Pad1.08x0.95mm_HandSolder
- R1: renamed from R3; footprint (none) -> Resistor_SMD:R_0805_2012Metric_Pad1.20x1.40mm_HandSolder
- R2: renamed from R4; footprint (none) -> Resistor_SMD:R_0805_2012Metric_Pad1.20x1.40mm_HandSolder
- SW1: value SW_Push -> LEFT_BTN
- SW2: value SW_Push -> RT_BTN
Connections:
- net GND is gone; now on an unnamed net: C1.1, U1.4 (GND), U2.10 (GND)
- net at C1.2, R1.1, U1.8 (VCC)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: now also SW1.2, SW2.2, BAT1.1 (Pin_1); no longer SW1.1, SW2.1
- net at U1.2 (XTAL1/PB3): now also SW1.1; no longer SW1.2
- net at U1.3 (XTAL2/PB4): now also SW2.1; no longer SW2.2
- net at U1.5 (AREF/PB0): now also R2.1; no longer R2.2
- net at U2.2 (RX): now also R2.2; no longer R2.1
- net at U2.6 (SPK_1): now also SPK1.2 (Pin_2)
- net at U2.8 (SPK_2): now also SPK1.1 (Pin_1)
- net at U2.7 (GND): now also BAT1.2 (Pin_2)
- no-connect marks 11 -> 10
Other:
- moved on the sheet: C1, R1, R2, U1, U2

Commit message: Do stuff in kicad
Parts:
- added H1, H2: MountingHole, MountingHole:MountingHole_3.2mm_M3, symbol Mechanical:MountingHole
- added H3, H4: AlignmentHole, MountingHole:MountingHole_2.5mm, symbol Mechanical:MountingHole
- SW1, SW2: footprint (none) -> Library:Keypad
- U2: value DFPLAYER MINI -> DFR0299; footprint (none) -> DFR0299:MODULE_DFR0299; symbol New_Library:DFPLAYER MINI -> DFR0299:DFR0299; AVAILABILITY (none) -> Unavailable; DESCRIPTION (none) -> Dfplayer - a Mini Mp3 Player; MF (none) -> DFRobot; MP (none) -> DFR0299; PACKAGE (none) -> None; PRICE (none) -> None
Connections:
- net at SPK1.1 (Pin_1): now also U2.6 (SPK1); no longer U2.8 (SPK_2)
- net at SPK1.2 (Pin_2): now also U2.8 (SPK2); no longer U2.6 (SPK_1)
- net VDD: now reaches BAT1.1 (Pin_1), C1.2, R1.1, SW1.2, SW2.2, U1.8 (VCC), U2.1 (VCC)
- net GND: now reaches BAT1.2 (Pin_2), C1.1, U1.4 (GND), U2.10 (GND__1), U2.7 (GND)
- net at U1.6 (PB1): now also U2.2 (RX); no longer U2.3 (TX)
- net at R2.2: now also U2.3 (TX); no longer U2.2 (RX)
- no-connect marks 10 -> 1
Other:
- moved on the sheet: SPK1, U2

Commit message: New footprint
Parts:
- C1: footprint Capacitor_SMD:C_0603_1608Metric_Pad1.08x0.95mm_HandSolder -> Capacitor_THT:C_Disc_D5.0mm_W2.5mm_P2.50mm; symbol Device:C -> Device:C_Small_US
- R1: footprint Resistor_SMD:R_0805_2012Metric_Pad1.20x1.40mm_HandSolder -> Resistor_THT:R_Axial_DIN0204_L3.6mm_D1.6mm_P5.08mm_Horizontal; symbol Device:R -> Device:R_US
- R2: footprint Resistor_SMD:R_0805_2012Metric_Pad1.20x1.40mm_HandSolder -> Resistor_THT:R_Axial_DIN0207_L6.3mm_D2.5mm_P7.62mm_Horizontal; symbol Device:R -> Device:R_US
- SW1, SW2: footprint Library:Keypad -> Library:Keypad 2
Changed lines of the file:
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@@
 	(paper "A4")
+	(junction
+		(at 66.04 68.58)
+		(diameter 0)
+		(color 0 0 0 0)
+	)
 	(junction
 		(at 125.73 85.09)
@@
 	)
 	(junction
-		(at 66.04 62.23)
-		(diameter 0)
-		(color 0 0 0 0)
-	)
-	(junction
 		(at 109.22 59.69)
-		(diameter 0)
-		(color 0 0 0 0)
-	)
-	(junction
-		(at 66.04 69.85)
 		(diameter 0)
 		(color 0 0 0 0)
@@
 	)
 	(junction
+		(at 66.04 63.5)
+		(diameter 0)
+		(color 0 0 0 0)
+	)
+	(junction
 		(at 71.12 59.69)
 		(diameter 0)
@@
 	(wire
 		(pts
-			(xy 62.23 67.31) (xy 62.23 69.85)
+			(xy 62.23 67.31) (xy 62.23 68.58)
 		)
 		(stroke
@@
 	(wire
 		(pts
-			(xy 62.23 62.23) (xy 66.04 62.23)
-		)
-		(stroke
-			(width 0)
-			(type default)
-			(color 255 0 0 1)
-		)
-	)
-	(wire
-		(pts
-			(xy 69.85 62.23) (xy 66.04 62.23)
+			(xy 62.23 63.5) (xy 66.04 63.5)
+		)
+		(stroke
+			(width 0)
+			(type default)
+			(color 255 0 0 1)
+		)
+	)
+	(wire
+		(pts
+			(xy 69.85 63.5) (xy 66.04 63.5)
 		)
 		(stroke
@@
 	(wire
 		(pts
-			(xy 69.85 69.85) (xy 66.04 69.85)
+			(xy 66.04 68.58) (xy 69.85 68.58)
 		)
 		(stroke
@@
 	(wire
 		(pts
+			(xy 66.04 68.58) (xy 66.04 74.93)
+		)
+		(stroke
+			(width 0)
+			(type default)
+			(color 0 0 0 1)
+		)
+	)
+	(wire
+		(pts
 			(xy 170.18 67.31) (xy 170.18 59.69)
 		)
@@
 	(wire
 		(pts
-			(xy 66.04 69.85) (xy 66.04 74.93)
+			(xy 113.03 78.74) (xy 113.03 74.93)
+		)
+		(stroke
+			(width 0)
+			(type default)
+		)
+	)
+	(wire
+		(pts
+			(xy 109.22 59.69) (xy 109.22 66.04)
+		)
+		(stroke
+			(width 0)
+			(type default)
+			(color 255 0 0 1)
+		)
+	)
+	(wire
+		(pts
+			(xy 109.22 99.06) (xy 109.22 101.6)
 		)
 		(stroke
@@
 	(wire
 		(pts
-			(xy 113.03 78.74) (xy 113.03 74.93)
-		)
-		(stroke
-			(width 0)
-			(type default)
-		)
-	)
-	(wire
-		(pts
-			(xy 109.22 59.69) (xy 109.22 66.04)
-		)
-		(stroke
-			(width 0)
-			(type default)
-			(color 255 0 0 1)
-		)
-	)
-	(wire
-		(pts
-			(xy 109.22 99.06) (xy 109.22 101.6)
-		)
-		(stroke
-			(width 0)
-			(type default)
-			(color 0 0 0 1)
-		)
-	)
-	(wire
-		(pts
 			(xy 113.03 74.93) (xy 144.78 74.93)
 		)
@@
 	(wire
 		(pts
-			(xy 62.23 62.23) (xy 62.23 64.77)
-		)
-		(stroke
-			(width 0)
-			(type default)
-			(color 255 0 0 1)
-		)
-	)
-	(wire
-		(pts
-			(xy 66.04 59.69) (xy 66.04 62.23)
+			(xy 62.23 63.5) (xy 62.23 64.77)
+		)
+		(stroke
+			(width 0)
+			(type default)
+			(color 255 0 0 1)
+		)
+	)
+	(wire
+		(pts
+			(xy 66.04 59.69) (xy 66.04 63.5)
 		)
 		(stroke
@@
 	(wire
 		(pts
-			(xy 62.23 69.85) (xy 66.04 69.85)
+			(xy 62.23 68.58) (xy 66.04 68.58)
 		)
 		(stroke
@@
 			)
 		)
-		(property "Footprint" "Library:Keypad"
+		(property "Footprint" "Library:Keypad 2"
 			(at 133.35 80.01 0)
 			(effects
@@
 	)
 	(symbol
-		(lib_id "Device:R")
+		(lib_id "Device:R_US")
 		(at 154.94 92.71 0)
 		(mirror x)
@@
 			)
 		)
-		(property "Footprint" "Resistor_SMD:R_0805_2012Metric_Pad1.20x1.40mm_HandSolder"
-			(at 153.162 92.71 90)
+		(property "Footprint" "Resistor_THT:R_Axial_DIN0204_L3.6mm_D1.6mm_P5.08mm_Horizontal"
+			(at 155.956 92.456 90)
 			(effects
 				(font
@@
 			)
 		)
-		(property "Description" "Resistor"
+		(property "Description" "Resistor, US symbol"
 			(at 154.94 92.71 0)
 			(effects
@@
 			)
 		)
-		(property "Footprint" "Library:Keypad"
+		(property "Footprint" "Library:Keypad 2"
 			(at 133.35 88.9 0)
 			(effects
@@
 	)
 	(symbol
-		(lib_id "Device:R")
+		(lib_id "Device:R_US")
 		(at 148.59 74.93 270)
 		(mirror x)
@@
 			)
 		)
-		(property "Footprint" "Resistor_SMD:R_0805_2012Metric_Pad1.20x1.40mm_HandSolder"
-			(at 148.59 76.708 90)
+		(property "Footprint" "Resistor_THT:R_Axial_DIN0207_L6.3mm_D2.5mm_P7.62mm_Horizontal"
+			(at 148.336 73.914 90)
 			(effects
 				(font
@@
 			)
 		)
-		(property "Description" "Resistor"
+		(property "Description" "Resistor, US symbol"
 			(at 148.59 74.93 0)
 			(effects
@@
 	)
 	(symbol
-		(lib_id "Device:C")
+		(lib_id "Device:C_Small_US")
 		(at 69.85 66.04 180)
 		(unit 1)
@@
 			)
 		)
-		(property "Footprint" "Capacitor_SMD:C_0603_1608Metric_Pad1.08x0.95mm_HandSolder"
-			(at 68.8848 62.23 0)
+		(property "Footprint" "Capacitor_THT:C_Disc_D5.0mm_W2.5mm_P2.50mm"
+			(at 69.85 66.04 0)
 			(effects
 				(font
@@
 			)
 		)
-		(property "Description" "Unpolarized capacitor"
+		(property "Description" "capacitor, small US symbol"
 			(at 69.85 66.04 0)
 			(effects
